File: pcb/temper.kicad_sch (KiCad schematic)
At the start: 41 parts, among them J2 nice_view, SW1 SW_PUSH, SW10 SW_PUSH, SW11 SW_PUSH, SW12 SW_PUSH, SW13 SW_PUSH, SW14 SW_PUSH, SW15 SW_PUSH, SW16 SW_PUSH, SW17 SW_PUSH, SW18 SW_PUSH, SW2 SW_PUSH, SW3 SW_PUSH, SW4 SW_PUSH, SW5 SW_PUSH, SW6 SW_PUSH, SW7 SW_PUSH, SW8 SW_PUSH, SW9 SW_PUSH, U1 nice_nano

Commit message: Convert switches to Choc v2 sockets
Parts:
- SW1, SW10, SW11, SW12, SW13, SW14, SW15, SW16, SW17, SW18, SW2, SW3, SW4, SW5, SW6, SW7, SW8, SW9: footprint dumta:Kailh_socket_PG1350_reversible -> dumta:Kailh_socket_Choc_V2_reversible
Changed lines of the file:
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@@
       (effects (font (size 1.27 1.27)))
     )
-    (property "Footprint" "dumta:Kailh_socket_PG1350_reversible" (at 49.53 43.815 0)
+    (property "Footprint" "dumta:Kailh_socket_Choc_V2_reversible" (at 49.53 43.815 0)
       (effects (font (size 1.27 1.27)) hide)
     )
@@
       (effects (font (size 1.27 1.27)))
     )
-    (property "Footprint" "dumta:Kailh_socket_PG1350_reversible" (at 67.31 43.815 0)
+    (property "Footprint" "dumta:Kailh_socket_Choc_V2_reversible" (at 67.31 43.815 0)
       (effects (font (size 1.27 1.27)) hide)
     )
@@
       (effects (font (size 1.27 1.27)))
     )
-    (property "Footprint" "dumta:Kailh_socket_PG1350_reversible" (at 85.09 43.815 0)
+    (property "Footprint" "dumta:Kailh_socket_Choc_V2_reversible" (at 85.09 43.815 0)
       (effects (font (size 1.27 1.27)) hide)
     )
@@
       (effects (font (size 1.27 1.27)))
     )
-    (property "Footprint" "dumta:Kailh_socket_PG1350_reversible" (at 102.87 43.815 0)
+    (property "Footprint" "dumta:Kailh_socket_Choc_V2_reversible" (at 102.87 43.815 0)
       (effects (font (size 1.27 1.27)) hide)
     )
@@
       (effects (font (size 1.27 1.27)))
     )
-    (property "Footprint" "dumta:Kailh_socket_PG1350_reversible" (at 120.65 43.815 0)
+    (property "Footprint" "dumta:Kailh_socket_Choc_V2_reversible" (at 120.65 43.815 0)
       (effects (font (size 1.27 1.27)) hide)
     )
@@
       (effects (font (size 1.27 1.27)))
     )
-    (property "Footprint" "dumta:Kailh_socket_PG1350_reversible" (at 49.53 59.055 0)
+    (property "Footprint" "dumta:Kailh_socket_Choc_V2_reversible" (at 49.53 59.055 0)
       (effects (font (size 1.27 1.27)) hide)
     )
@@
       (effects (font (size 1.27 1.27)))
     )
-    (property "Footprint" "dumta:Kailh_socket_PG1350_reversible" (at 67.31 59.055 0)
+    (property "Footprint" "dumta:Kailh_socket_Choc_V2_reversible" (at 67.31 59.055 0)
       (effects (font (size 1.27 1.27)) hide)
     )
@@
       (effects (font (size 1.27 1.27)))
     )
-    (property "Footprint" "dumta:Kailh_socket_PG1350_reversible" (at 85.09 59.055 0)
+    (property "Footprint" "dumta:Kailh_socket_Choc_V2_reversible" (at 85.09 59.055 0)
       (effects (font (size 1.27 1.27)) hide)
     )
@@
       (effects (font (size 1.27 1.27)))
     )
-    (property "Footprint" "dumta:Kailh_socket_PG1350_reversible" (at 102.87 59.055 0)
+    (property "Footprint" "dumta:Kailh_socket_Choc_V2_reversible" (at 102.87 59.055 0)
       (effects (font (size 1.27 1.27)) hide)
     )
@@
       (effects (font (size 1.27 1.27)))
     )
-    (property "Footprint" "dumta:Kailh_socket_PG1350_reversible" (at 120.65 59.055 0)
+    (property "Footprint" "dumta:Kailh_socket_Choc_V2_reversible" (at 120.65 59.055 0)
       (effects (font (size 1.27 1.27)) hide)
     )
@@
       (effects (font (size 1.27 1.27)))
     )
-    (property "Footprint" "dumta:Kailh_socket_PG1350_reversible" (at 49.53 74.295 0)
+    (property "Footprint" "dumta:Kailh_socket_Choc_V2_reversible" (at 49.53 74.295 0)
       (effects (font (size 1.27 1.27)) hide)
     )
@@
       (effects (font (size 1.27 1.27)))
     )
-    (property "Footprint" "dumta:Kailh_socket_PG1350_reversible" (at 67.31 74.295 0)
+    (property "Footprint" "dumta:Kailh_socket_Choc_V2_reversible" (at 67.31 74.295 0)
       (effects (font (size 1.27 1.27)) hide)
     )
@@
       (effects (font (size 1.27 1.27)))
     )
-    (property "Footprint" "dumta:Kailh_socket_PG1350_reversible" (at 85.09 74.295 0)
+    (property "Footprint" "dumta:Kailh_socket_Choc_V2_reversible" (at 85.09 74.295 0)
       (effects (font (size 1.27 1.27)) hide)
     )
@@
       (effects (font (size 1.27 1.27)))
     )
-    (property "Footprint" "dumta:Kailh_socket_PG1350_reversible" (at 102.87 74.295 0)
+    (property "Footprint" "dumta:Kailh_socket_Choc_V2_reversible" (at 102.87 74.295 0)
       (effects (font (size 1.27 1.27)) hide)
     )
@@
       (effects (font (size 1.27 1.27)))
     )
-    (property "Footprint" "dumta:Kailh_socket_PG1350_reversible" (at 120.65 74.295 0)
+    (property "Footprint" "dumta:Kailh_socket_Choc_V2_reversible" (at 120.65 74.295 0)
       (effects (font (size 1.27 1.27)) hide)
     )
@@
       (effects (font (size 1.27 1.27)))
     )
-    (property "Footprint" "dumta:Kailh_socket_PG1350_reversible" (at 105.41 104.14 0)
+    (property "Footprint" "dumta:Kailh_socket_Choc_V2_reversible" (at 105.41 104.14 0)
       (effects (font (size 1.27 1.27)) hide)
     )
@@
       (effects (font (size 1.27 1.27)))
     )
-    (property "Footprint" "dumta:Kailh_socket_PG1350_reversible" (at 120.65 89.535 0)
+    (property "Footprint" "dumta:Kailh_socket_Choc_V2_reversible" (at 120.65 89.535 0)
       (effects (font (size 1.27 1.27)) hide)
     )
@@
       (effects (font (size 1.27 1.27)))
     )
-    (property "Footprint" "dumta:Kailh_socket_PG1350_reversible" (at 83.82 97.79 0)
-      (effects (font (size 1.27 1.27)) hide)
-    )
+    (property "Footprint" "dumta:Kailh_socket_Choc_V2_reversible" (at 83.82 97.79 0)
+      (effects (font (size 1.27 1.27)) hide)
+    )

Commit message: Clean up Choc v2 manufacturing files
Parts:
- SW1: footprint dumta:Kailh_socket_Choc_V2_reversible -> dumta:Kailh_socket_Choc_V2_reversible_edge_left_SW1
- SW11: footprint dumta:Kailh_socket_Choc_V2_reversible -> dumta:Kailh_socket_Choc_V2_reversible_edge_both_SW11
- SW16: footprint dumta:Kailh_socket_Choc_V2_reversible -> dumta:Kailh_socket_Choc_V2_reversible_rot180_SW16
- SW17: footprint dumta:Kailh_socket_Choc_V2_reversible -> dumta:Kailh_socket_Choc_V2_reversible_rot165_SW17
- SW18: footprint dumta:Kailh_socket_Choc_V2_reversible -> dumta:Kailh_socket_Choc_V2_reversible_rot240_SW18
- SW2: footprint dumta:Kailh_socket_Choc_V2_reversible -> dumta:Kailh_socket_Choc_V2_reversible_edge_left_SW2
- SW6: footprint dumta:Kailh_socket_Choc_V2_reversible -> dumta:Kailh_socket_Choc_V2_reversible_edge_left_SW6
Changed lines of the file:
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@@
       (effects (font (size 1.27 1.27)))
     )
-    (property "Footprint" "dumta:Kailh_socket_Choc_V2_reversible" (at 49.53 43.815 0)
+    (property "Footprint" "dumta:Kailh_socket_Choc_V2_reversible_edge_left_SW1" (at 49.53 43.815 0)
       (effects (font (size 1.27 1.27)) hide)
     )
@@
       (effects (font (size 1.27 1.27)))
     )
-    (property "Footprint" "dumta:Kailh_socket_Choc_V2_reversible" (at 67.31 43.815 0)
+    (property "Footprint" "dumta:Kailh_socket_Choc_V2_reversible_edge_left_SW2" (at 67.31 43.815 0)
       (effects (font (size 1.27 1.27)) hide)
     )
@@
       (effects (font (size 1.27 1.27)))
     )
-    (property "Footprint" "dumta:Kailh_socket_Choc_V2_reversible" (at 49.53 59.055 0)
+    (property "Footprint" "dumta:Kailh_socket_Choc_V2_reversible_edge_left_SW6" (at 49.53 59.055 0)
       (effects (font (size 1.27 1.27)) hide)
     )
@@
       (effects (font (size 1.27 1.27)))
     )
-    (property "Footprint" "dumta:Kailh_socket_Choc_V2_reversible" (at 49.53 74.295 0)
+    (property "Footprint" "dumta:Kailh_socket_Choc_V2_reversible_edge_both_SW11" (at 49.53 74.295 0)
       (effects (font (size 1.27 1.27)) hide)
     )
@@
       (effects (font (size 1.27 1.27)))
     )
-    (property "Footprint" "dumta:Kailh_socket_Choc_V2_reversible" (at 105.41 104.14 0)
+    (property "Footprint" "dumta:Kailh_socket_Choc_V2_reversible_rot165_SW17" (at 105.41 104.14 0)
       (effects (font (size 1.27 1.27)) hide)
     )
@@
       (effects (font (size 1.27 1.27)))
     )
-    (property "Footprint" "dumta:Kailh_socket_Choc_V2_reversible" (at 120.65 89.535 0)
+    (property "Footprint" "dumta:Kailh_socket_Choc_V2_reversible_rot240_SW18" (at 120.65 89.535 0)
       (effects (font (size 1.27 1.27)) hide)
     )
@@
       (effects (font (size 1.27 1.27)))
     )
-    (property "Footprint" "dumta:Kailh_socket_Choc_V2_reversible" (at 83.82 97.79 0)
-      (effects (font (size 1.27 1.27)) hide)
-    )
+    (property "Footprint" "dumta:Kailh_socket_Choc_V2_reversible_rot180_SW16" (at 83.82 97.79 0)
+      (effects (font (size 1.27 1.27)) hide)
+    )
